File: hardware/kicad-integrated/Surfshot_Integrated.kicad_sch (KiCad schematic)
At the start: 35 parts, among them J1 PROTECTED_CELL, J2 UART_3V3_LEVEL, J3 LORA_EXPANSION, J4 MOTOR_A, J5 MOTOR_B, SW1 RESET, SW2 BOOT, U1 ESP32-WROOM-32E-N4, U2 TPS62162DSG, U3 ULN2003A, U4 ULN2003A

Commit message: Redraw B0.1 with directly wired local circuit blocks: Surfshot_Integrated.kicad_sch
Connections:
- net A_COIL1: no longer names the net of J4.2 (Pin_2), U3.16 (O1)
- net A_COIL2: no longer names the net of J4.3 (Pin_3), U3.15 (O2)
- net A_COIL3: no longer names the net of J4.4 (Pin_4), U3.14 (O3)
- net A_COIL4: no longer names the net of J4.5 (Pin_5), U3.13 (O4)
- net BAT_RAW: no longer names the net of F1.1, J1.1 (Pin_1)
- net B_COIL1: no longer names the net of J5.2 (Pin_2), U4.16 (O1)
- net B_COIL2: no longer names the net of J5.3 (Pin_3), U4.15 (O2)
- net B_COIL3: no longer names the net of J5.4 (Pin_4), U4.14 (O3)
- net B_COIL4: no longer names the net of J5.5 (Pin_5), U4.13 (O4)
- net SW_3V3: no longer names the net of L1.1, U2.7 (SW)
Other:
- removed sheet On-board 5V and 12V converters
- added sheet 5 V / 12 V boost converters (Power.kicad_sch)
- note added: "18650 INPUT / EXTERNAL PROTECTION"
- note added: "3.3 V LOGIC SUPPLY"
- note added: "3.3 V UART only. Hold BOOT, tap RESET. Power from battery; no adapter power connection."
- note added: "B0.1: drawing readability revision; electrical connectivity unchanged. SuperMini socket conversion pending actual board pinout."
- note added: "BATTERY ADC"
- note added: "CONTROLLER / LOCAL BYPASS"
- note added: "J pin 1: common; 2-5: coils. Verify harness order."
- note added: "MOTOR A / +5V_M"
- note added: "MOTOR B / +12V_M"
- note added: "PG -> ESP_EN. Keep input/output current loops short."
- note added: "Power targets: 5 V / 1 A total, 12 V / 0.6 A. Not measured continuous output ratings."
- note added: "RESET / BOOT"
- note added: "SURFSHOT / CONTROLLER AND MOTOR DRIVERS"
- note added: "Single 18650; cell/BMS current rating pending. F1 and connector selection provisional."
- note added: "WROOM version retained; S3 SuperMini pinout not yet supplied. Motor GPIOs: A = 13,14,16,17; B = 25,26,27,32."
- note removed: "3.0-4.2 V design range. External charger/BMS. Fuse, connector and wire ratings require pack data. External main disconnect; no reverse-polarity circuit."
- note removed: "3.3 V LOGIC SUPPLY / 1 A CLASS"
- note removed: "A MOTOR / +5V_M"
- note removed: "B MOTOR / +12V_M"
- note removed: "BATTERY INPUT"
- note removed: "Direct PCB circuit: 1-cell protected battery -> on-board 5 V / 12 V boost -> motors; 5 V -> 3.3 V buck -> ESP32"
- note removed: "ESP32-WROOM-32E-N4 / SOLDERED MODULE"
- note removed: "External USB-UART, 3.3 V logic only. Power from battery, not serial adapter. Hold BOOT, tap RESET to download."
- note removed: "J pin 1 = common; 2-5 = coil ends. Verify harness order and phase sequence. Two-phase stepping maximum for initial test."
- note removed: "Motor GPIOs: A = 13,14,16,17; B = 25,26,27,32. Module antenna must face board edge / copper keepout. Use N4 (no PSRAM); do not substitute R2 variant blindly."
- note removed: "PG open drain holds ESP_EN low during undervoltage. Short SW loop; Kelvin VOS from output capacitor."
- note removed: "RESET / BOOT / BATTERY MONITOR"
- note removed: "SURFSHOT / INTEGRATED CONTROLLER - REV B0"
- note removed: "Targets, not verified ratings: 5 V rail: 1.0 A total (motor + logic) 12 V rail: 0.6 A motor 3 V battery current: approx. 4.8 A at 85% efficiency."
- title: Surfshot integrated controller / logic and motor drive -> Surfshot / controller and motor drive
