File: hardware/kicad-integrated/Power.kicad_sch (KiCad schematic)
At the start: 32 parts, among them U5 TPS61089RNR, U6 TPS61089RNR

Commit message: Redraw B0.1 with directly wired local circuit blocks: Power.kicad_sch
Parts:
- removed U5, U6: TPS61089RNR, Package_DFN_QFN:Texas_VQFN-RNR0011A-11, symbol Regulator_Switching:TPS61089
- added U5, U6: TPS61089RNR, Package_DFN_QFN:Texas_VQFN-RNR0011A-11, symbol Surfshot:TPS61089_Logical
Connections:
- net +12V_M: now also U6.6 (VOUT)
- net +5V_M: now also U5.6 (VOUT)
- net GND: now also U5.5 (GND), U6.5 (GND)
- net VBAT: now also U5.7 (EN), U5.9 (VIN), U6.7 (EN), U6.9 (VIN)
- net P12_BOOT: no longer names the net of C25.1
- net P12_BOOT: now also U6.10 (BOOT)
- net P12_COMP: no longer names the net of C24.1, R22.1
- net P12_COMP: now also U6.4 (COMP)
- net P12_FB: no longer names the net of R20.2, R21.1
- net P12_FB: now also U6.3 (FB)
- net P12_FSW: no longer names the net of R23.2
- net P12_FSW: now also U6.1 (FSW)
- net P12_ILIM: no longer names the net of R24.1
- net P12_ILIM: now also U6.8 (ILIM)
- net P12_RC: no longer names the net of C23.1, R22.2
- net P12_SW: no longer names the net of C25.2, L3.2, R23.1
- net P12_SW: now also U6.11 (SW)
- net P12_VCC: no longer names the net of C26.1
- net P12_VCC: now also U6.2 (VCC)
- net P5_BOOT: no longer names the net of C16.1
- net P5_BOOT: now also U5.10 (BOOT)
- net P5_COMP: no longer names the net of C15.1, R17.1
- net P5_COMP: now also U5.4 (COMP)
- net P5_FB: no longer names the net of R15.2, R16.1
- net P5_FB: now also U5.3 (FB)
- net P5_FSW: no longer names the net of R18.2
- net P5_FSW: now also U5.1 (FSW)
- net P5_ILIM: no longer names the net of R19.1
- net P5_ILIM: now also U5.8 (ILIM)
- net P5_RC: no longer names the net of C14.1, R17.2
- net P5_SW: no longer names the net of C16.2, L2.2, R18.1
- net P5_SW: now also U5.11 (SW)
- net P5_VCC: no longer names the net of C17.1
- net P5_VCC: now also U5.2 (VCC)
Other:
- note added: "12 V / 0.6 A MOTOR - provisional targets"
- note added: "5 V / 1.0 A TOTAL - provisional targets"
- note added: "Calculated compensation; no hardware/thermal validation yet. EN-off does not disconnect output. Input: protected single cell. PCB outline target approx. 80 x 50 mm; layout not started."
- note added: "SURFSHOT / ON-BOARD BOOST CONVERTERS"
- note added: "Solid wires show local connections. Only VBAT, output rails and GND cross functional blocks."
- note added: "VIN / VCC / BOOT bypass: place at IC. Output bank: >=40uF effective after DC bias. FB / COMP: keep away from switching copper."
- note removed: "12 V / 0.6 A - DESIGN TARGET ONLY"
- note removed: "3.0-4.2 V input. Compensation values are calculated starting points; verify loop response on the actual PCB."
- note removed: "5 V / 1.0 A total - DESIGN TARGET ONLY"
- note removed: "FSW resistor connects to SW, not GND. BOOT capacitor connects to SW, not GND. VCC is local bypass only; never tie it to +3V3."
- note removed: "No charging IC or cell protection on this sheet. Use protected battery input. Disable motor coils below 3.2 V in firmware; battery BMS supplies hardware undervoltage cutoff. No load/transient/thermal validation yet. Use 4-layer PCB with solid GND for the next layout stage."
- note removed: "ON-BOARD POWER / TWO TPS61089 BOOST CONVERTERS"
- note removed: "Place VIN bypass, VCC bypass and BOOT cap at IC. Place output ceramics at VOUT/GND; minimize hot loop. Keep FB/COMP away from SW copper and RF antenna. Output capacitance assumption: >=40uF effective after DC bias. EN off does not isolate output: input can pass through body diode."
- title: Surfshot integrated controller / 5V and 12V boosts -> Surfshot / 5 V and 12 V power stages
